File: _saved_midiPedalboard_Perfboard.sch (KiCad schematic (older format))
At the start: 43 parts, among them J1 wire, J10 wire, J11 wire, J12 wire, J13 wire, J14 wire, J15 MIDI_4, J16 MIDI_5, J17 MIDI_4, J18 MIDI_2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

Commit message: add a second exp pedal input
Parts:
- added Jr11, Js11, Jt11: wire, Connector_Wire:SolderWirePad_1x01_Drill0.8mm, symbol Connector:Conn_01x01_Female
- added R6: 100, Resistor_THT:R_Axial_DIN0207_L6.3mm_D2.5mm_P2.54mm_Vertical, symbol Device:R_Small
Connections:
- net GND: now also Js11.1 (Pin_1)
- net VCC: now also R6.2
- net exp_2: now reaches U1.A5
- net exp_2: now also Jt11.1 (Pin_1)
- new net: Jr11.1 (Pin_1), R6.1
- no-connect marks 11 -> 10
Other:
- moved on the sheet: Jr10, Js10, R5
Changed lines of the file:
@@
 	-1   0    0    1
 $EndComp
-NoConn ~ 5900 3500
 NoConn ~ 5900 4100
 NoConn ~ 5900 4200
@@
 L Connector:Conn_01x01_Female Jr10
 U 1 1 5CAF6041
-P 7250 3050
-F 0 "Jr10" H 7300 3100 50  0000 C CNN
-F 1 "wire" H 7150 3100 50  0000 C CNN
-F 2 "Connector_Wire:SolderWirePad_1x01_Drill0.8mm" H 7250 3050 50  0001 C CNN
-F 3 "~" H 7250 3050 50  0001 C CNN
-	1    7250 3050
+P 6750 2900
+F 0 "Jr10" H 6800 2950 50  0000 C CNN
+F 1 "wire" H 6650 2950 50  0000 C CNN
+F 2 "Connector_Wire:SolderWirePad_1x01_Drill0.8mm" H 6750 2900 50  0001 C CNN
+F 3 "~" H 6750 2900 50  0001 C CNN
+	1    6750 2900
 	1    0    0    -1
 $EndComp
@@
 L Connector:Conn_01x01_Female Js10
 U 1 1 5CAF60E1
-P 7250 3250
-F 0 "Js10" H 7300 3300 50  0000 C CNN
-F 1 "wire" H 7150 3300 50  0000 C CNN
-F 2 "Connector_Wire:SolderWirePad_1x01_Drill0.8mm" H 7250 3250 50  0001 C CNN
-F 3 "~" H 7250 3250 50  0001 C CNN
-	1    7250 3250
+P 6750 3000
+F 0 "Js10" H 6800 3050 50  0000 C CNN
+F 1 "wire" H 6650 3050 50  0000 C CNN
+F 2 "Connector_Wire:SolderWirePad_1x01_Drill0.8mm" H 6750 3000 50  0001 C CNN
+F 3 "~" H 6750 3000 50  0001 C CNN
+	1    6750 3000
 	1    0    0    -1
 $EndComp
@@
 L Device:R_Small R5
 U 1 1 5CAF65EA
-P 7000 2900
-F 0 "R5" V 7000 2900 50  0000 C CNN
-F 1 "100" V 6895 2900 50  0001 C CNN
-F 2 "Resistor_THT:R_Axial_DIN0207_L6.3mm_D2.5mm_P2.54mm_Vertical" H 7000 2900 50  0001 C CNN
-F 3 "~" H 7000 2900 50  0001 C CNN
-	1    7000 2900
+P 6500 2750
+F 0 "R5" V 6500 2750 50  0000 C CNN
+F 1 "100" V 6395 2750 50  0001 C CNN
+F 2 "Resistor_THT:R_Axial_DIN0207_L6.3mm_D2.5mm_P2.54mm_Vertical" H 6500 2750 50  0001 C CNN
+F 3 "~" H 6500 2750 50  0001 C CNN
+	1    6500 2750
 	-1   0    0    1
 $EndComp
@@
 L power:VCC #PWR0109
 U 1 1 5CAF680A
-P 7000 2700
-F 0 "#PWR0109" H 7000 2550 50  0001 C CNN
-F 1 "VCC" H 7017 2873 50  0000 C CNN
-F 2 "" H 7000 2700 50  0001 C CNN
-F 3 "" H 7000 2700 50  0001 C CNN
-	1    7000 2700
-	1    0    0    -1
-$EndComp
-Wire Wire Line
-	7000 2700 7000 2800
-Wire Wire Line
-	7000 3000 7000 3050
-Wire Wire Line
-	7000 3050 7050 3050
-Wire Wire Line
-	7050 3250 7000 3250
-Wire Wire Line
-	7000 3250 7000 3300
+P 6500 2550
+F 0 "#PWR0109" H 6500 2400 50  0001 C CNN
+F 1 "VCC" H 6517 2723 50  0000 C CNN
+F 2 "" H 6500 2550 50  0001 C CNN
+F 3 "" H 6500 2550 50  0001 C CNN
+	1    6500 2550
+	1    0    0    -1
+$EndComp
+Wire Wire Line
+	6500 2550 6500 2650
+Wire Wire Line
+	6500 2850 6500 2900
+Wire Wire Line
+	6500 2900 6550 2900
+Wire Wire Line
+	6550 3000 6500 3000
+Wire Wire Line
+	6500 3000 6500 3050
 $Comp
 L power:GND #PWR0110
 U 1 1 5CAFA231
-P 7000 3300
-F 0 "#PWR0110" H 7000 3050 50  0001 C CNN
-F 1 "GND" H 7005 3127 50  0000 C CNN
-F 2 "" H 7000 3300 50  0001 C CNN
-F 3 "" H 7000 3300 50  0001 C CNN
-	1    7000 3300
+P 6500 3050
+F 0 "#PWR0110" H 6500 2800 50  0001 C CNN
+F 1 "GND" H 6505 2877 50  0000 C CNN
+F 2 "" H 6500 3050 50  0001 C CNN
+F 3 "" H 6500 3050 50  0001 C CNN
+	1    6500 3050
 	1    0    0    -1
 $EndComp
@@
 	1    0    0    -1
 $EndComp
+Wire Wire Line
+	5900 3500 6300 3500
+Text Label 6300 3500 2    50   ~ 0
+exp_2
+$Comp
+L Connector:Conn_01x01_Female Jt11
+U 1 1 5CCAFC10
+P 6500 3500
+F 0 "Jt11" H 6550 3550 50  0000 C CNN
+F 1 "wire" H 6400 3550 50  0000 C CNN
+F 2 "Connector_Wire:SolderWirePad_1x01_Drill0.8mm" H 6500 3500 50  0001 C CNN
+F 3 "~" H 6500 3500 50  0001 C CNN
+	1    6500 3500
+	1    0    0    -1
+$EndComp
+$Comp
+L Connector:Conn_01x01_Female Jr11
+U 1 1 5CCBBBC1
+P 7250 2900
+F 0 "Jr11" H 7300 2950 50  0000 C CNN
+F 1 "wire" H 7150 2950 50  0000 C CNN
+F 2 "Connector_Wire:SolderWirePad_1x01_Drill0.8mm" H 7250 2900 50  0001 C CNN
+F 3 "~" H 7250 2900 50  0001 C CNN
+	1    7250 2900
+	1    0    0    -1
+$EndComp
+$Comp
+L Connector:Conn_01x01_Female Js11
+U 1 1 5CCBBBC8
+P 7250 3000
+F 0 "Js11" H 7300 3050 50  0000 C CNN
+F 1 "wire" H 7150 3050 50  0000 C CNN
+F 2 "Connector_Wire:SolderWirePad_1x01_Drill0.8mm" H 7250 3000 50  0001 C CNN
+F 3 "~" H 7250 3000 50  0001 C CNN
+	1    7250 3000
+	1    0    0    -1
+$EndComp
+$Comp
+L Device:R_Small R6
+U 1 1 5CCBBBCF
+P 7000 2750
+F 0 "R6" V 7000 2750 50  0000 C CNN
+F 1 "100" V 6895 2750 50  0001 C CNN
+F 2 "Resistor_THT:R_Axial_DIN0207_L6.3mm_D2.5mm_P2.54mm_Vertical" H 7000 2750 50  0001 C CNN
+F 3 "~" H 7000 2750 50  0001 C CNN
+	1    7000 2750
+	-1   0    0    1
+$EndComp
+$Comp
+L power:VCC #PWR0101
+U 1 1 5CCBBBD6
+P 7000 2550
+F 0 "#PWR0101" H 7000 2400 50  0001 C CNN
+F 1 "VCC" H 7017 2723 50  0000 C CNN
+F 2 "" H 7000 2550 50  0001 C CNN
+F 3 "" H 7000 2550 50  0001 C CNN
+	1    7000 2550
+	1    0    0    -1
+$EndComp
+Wire Wire Line
+	7000 2550 7000 2650
+Wire Wire Line
+	7000 2850 7000 2900
+Wire Wire Line
+	7000 2900 7050 2900
+Wire Wire Line
+	7050 3000 7000 3000
+Wire Wire Line
+	7000 3000 7000 3050
+$Comp
+L power:GND #PWR0111
+U 1 1 5CCBBBE1
+P 7000 3050
+F 0 "#PWR0111" H 7000 2800 50  0001 C CNN
+F 1 "GND" H 7005 2877 50  0000 C CNN
+F 2 "" H 7000 3050 50  0001 C CNN
+F 3 "" H 7000 3050 50  0001 C CNN
+	1    7000 3050
+	1    0    0    -1
+$EndComp
